File: hardware/pcb/keypad.sch (KiCad schematic (older format))
At the start: 13 parts

Commit message: vbh: pcb layout
Parts:
- SW_A1, SW_B1, SW_DOWN1, SW_LEFT1, SW_RIGHT1, SW_SELECT1, SW_START1, SW_UP1: footprint (none) -> footprint:Contact_4mm
Changed lines of the file:
@@
 F 0 "SW_LEFT1" H 4000 3693 50  0000 C CNN
 F 1 "SW_Push" H 4000 3694 50  0001 C CNN
-F 2 "" H 4000 3700 50  0001 C CNN
+F 2 "footprint:Contact_4mm" H 4000 3700 50  0001 C CNN
 F 3 "~" H 4000 3700 50  0001 C CNN
 	1    4000 3500
@@
 F 0 "SW_UP1" H 4800 3293 50  0000 C CNN
 F 1 "SW_Push" H 4800 3294 50  0001 C CNN
-F 2 "" H 4800 3300 50  0001 C CNN
+F 2 "footprint:Contact_4mm" H 4800 3300 50  0001 C CNN
 F 3 "~" H 4800 3300 50  0001 C CNN
 	1    4800 3100
@@
 F 0 "SW_RIGHT1" H 5600 3693 50  0000 C CNN
 F 1 "SW_Push" H 5600 3694 50  0001 C CNN
-F 2 "" H 5600 3700 50  0001 C CNN
+F 2 "footprint:Contact_4mm" H 5600 3700 50  0001 C CNN
 F 3 "~" H 5600 3700 50  0001 C CNN
 	1    5600 3500
@@
 F 0 "SW_DOWN1" H 4800 4193 50  0000 C CNN
 F 1 "SW_Push" H 4800 4194 50  0001 C CNN
-F 2 "" H 4800 4200 50  0001 C CNN
+F 2 "footprint:Contact_4mm" H 4800 4200 50  0001 C CNN
 F 3 "~" H 4800 4200 50  0001 C CNN
 	1    4800 4000
@@
 F 0 "SW_B1" H 7300 4193 50  0000 C CNN
 F 1 "SW_Push" H 7300 4194 50  0001 C CNN
-F 2 "" H 7300 4200 50  0001 C CNN
+F 2 "footprint:Contact_4mm" H 7300 4200 50  0001 C CNN
 F 3 "~" H 7300 4200 50  0001 C CNN
 	1    7300 4000
@@
 F 0 "SW_A1" H 8300 3993 50  0000 C CNN
 F 1 "SW_Push" H 8300 3994 50  0001 C CNN
-F 2 "" H 8300 4000 50  0001 C CNN
+F 2 "footprint:Contact_4mm" H 8300 4000 50  0001 C CNN
 F 3 "~" H 8300 4000 50  0001 C CNN
 	1    8300 3800
@@
 F 0 "SW_START1" H 7300 3293 50  0000 C CNN
 F 1 "SW_Push" H 7300 3294 50  0001 C CNN
-F 2 "" H 7300 3300 50  0001 C CNN
+F 2 "footprint:Contact_4mm" H 7300 3300 50  0001 C CNN
 F 3 "~" H 7300 3300 50  0001 C CNN
 	1    7300 3100
@@
 F 0 "SW_SELECT1" H 8300 3293 50  0000 C CNN
 F 1 "SW_Push" H 8300 3294 50  0001 C CNN
-F 2 "" H 8300 3300 50  0001 C CNN
+F 2 "footprint:Contact_4mm" H 8300 3300 50  0001 C CNN
 F 3 "~" H 8300 3300 50  0001 C CNN
 	1    8300 3100
