File: hardware/pcb/lcd.sch (KiCad schematic (older format))
At the start: 26 parts, among them J400 Conn_02x10_Top_Bottom_Mountin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, U400 TC358778, U401 TPS65631W, U402 AP2127K-3.0

Commit message: vbh: pcb layout
Parts:
- U401: footprint Package_DFN_QFN:DFN-8-1EP_3x2mm_P0.5mm_EP1.36x1.46mm -> Package_DFN_QFN:DFN-10-1EP_3x3mm_P0.5mm_EP1.55x2.48mm
Changed lines of the file:
@@
 F 0 "U401" H 7900 4565 50  0000 C CNN
 F 1 "TPS65631W" H 7900 4474 50  0000 C CNN
-F 2 "Package_DFN_QFN:DFN-8-1EP_3x2mm_P0.5mm_EP1.36x1.46mm" H 7900 4500 50  0001 C CNN
+F 2 "Package_DFN_QFN:DFN-10-1EP_3x3mm_P0.5mm_EP1.55x2.48mm" H 7900 4500 50  0001 C CNN
 F 3 "" H 7900 4500 50  0001 C CNN
 	1    7900 4500
