File: hardware/pcb/microsd.sch (KiCad schematic (older format))
At the start: 7 parts

Commit message: vbh: pcb layout
Parts:
- MICRO_SD300: footprint footprints:TFC-WPAPR-08 -> footprint:TFC-WPAPR-08
- R600, R601, R602: footprint Resistor_SMD:R_0603_1608Metric -> Resistor_SMD:R_0402_1005Metric
Changed lines of the file:
@@
 F 0 "MICRO_SD300" H 7028 4603 60  0000 L CNN
 F 1 "MICRO_SD(TFC-WPAPR-08)" H 7028 4497 60  0000 L CNN
-F 2 "footprints:TFC-WPAPR-08" H 6950 4500 60  0001 C CNN
+F 2 "footprint:TFC-WPAPR-08" H 6950 4500 60  0001 C CNN
 F 3 "" H 6950 4500 60  0001 C CNN
 	1    6700 4500
@@
 F 0 "R601" H 5470 3696 50  0000 L CNN
 F 1 "10K" H 5470 3605 50  0000 L CNN
-F 2 "Resistor_SMD:R_0603_1608Metric" V 5330 3650 50  0001 C CNN
+F 2 "Resistor_SMD:R_0402_1005Metric" V 5330 3650 50  0001 C CNN
 F 3 "~" H 5400 3650 50  0001 C CNN
 	1    5400 3650
@@
 F 0 "R602" H 4970 3696 50  0000 L CNN
 F 1 "10K" H 4970 3605 50  0000 L CNN
-F 2 "Resistor_SMD:R_0603_1608Metric" V 4830 3650 50  0001 C CNN
+F 2 "Resistor_SMD:R_0402_1005Metric" V 4830 3650 50  0001 C CNN
 F 3 "~" H 4900 3650 50  0001 C CNN
 	1    4900 3650
@@
 F 0 "R600" V 5600 4000 50  0000 C CNN
 F 1 "33R" V 5600 4400 50  0000 C CNN
-F 2 "Resistor_SMD:R_0603_1608Metric" V 5580 4200 50  0001 C CNN
+F 2 "Resistor_SMD:R_0402_1005Metric" V 5580 4200 50  0001 C CNN
 F 3 "~" H 5650 4200 50  0001 C CNN
 	1    5650 4200
