File: hardware/pcb/power.sch (KiCad schematic (older format))
At the start: 47 parts, among them U1 AXP209, U100 XC6SLX16-FTG256, U2 SY8008

Commit message: vbh: pcb layout
Parts:
- added BAT1: Conn_01x03, footprint:BC-15-3P, symbol Connector_Generic:Conn_01x03
- C20: value 4.7uF -> 100nF; footprint Capacitor_SMD:C_0603_1608Metric -> Capacitor_SMD:C_0402_1005Metric
- R5: footprint Resistor_SMD:R_0805_2012Metric -> Resistor_SMD:R_0603_1608Metric
Connections:
- net +BATT: now also BAT1.1 (Pin_1)
- net GND: now also BAT1.3 (Pin_3)
- net TS: now reaches U1.37 (TS)
- net TS: now also BAT1.2 (Pin_2)
- no-connect marks 7 -> 6
Changed lines of the file:
@@
 F 0 "R5" V 4800 3700 50  0000 C CNN
 F 1 "1R" V 4800 4100 50  0000 C CNN
-F 2 "Resistor_SMD:R_0805_2012Metric" V 4780 3900 50  0001 C CNN
+F 2 "Resistor_SMD:R_0603_1608Metric" V 4780 3900 50  0001 C CNN
 F 3 "~" H 4850 3900 50  0001 C CNN
 	1    4850 3900
@@
 P 5550 4200
 F 0 "C20" V 5500 4050 50  0000 C CNN
-F 1 "4.7uF" V 5500 4350 50  0000 C CNN
-F 2 "Capacitor_SMD:C_0603_1608Metric" H 5588 4050 50  0001 C CNN
+F 1 "100nF" V 5500 4350 50  0000 C CNN
+F 2 "Capacitor_SMD:C_0402_1005Metric" H 5588 4050 50  0001 C CNN
 F 3 "~" H 5550 4200 50  0001 C CNN
 	1    5550 4200
@@
 NoConn ~ 2900 3500
 NoConn ~ 2900 3400
-NoConn ~ 2900 3000
 NoConn ~ 2900 2600
 NoConn ~ 2900 2500
@@
 	4100 6900 4100 6800
 Connection ~ 4600 6900
+$Comp
+L Connector_Generic:Conn_01x03 BAT1
+U 1 1 5E15F002
+P 2700 1900
+F 0 "BAT1" H 2780 1942 50  0000 L CNN
+F 1 "Conn_01x03" H 2780 1851 50  0000 L CNN
+F 2 "footprint:BC-15-3P" H 2700 1900 50  0001 C CNN
+F 3 "~" H 2700 1900 50  0001 C CNN
+	1    2700 1900
+	1    0    0    -1
+$EndComp
+Text Label 2300 1900 0    50   ~ 0
+TS
+Text Label 2700 3000 0    50   ~ 0
+TS
+Wire Wire Line
+	2700 3000 2900 3000
+$Comp
+L power:GND #PWR0102
+U 1 1 5E172A4A
+P 2400 2000
+F 0 "#PWR0102" H 2400 1750 50  0001 C CNN
+F 1 "GND" H 2405 1827 50  0000 C CNN
+F 2 "" H 2400 2000 50  0001 C CNN
+F 3 "" H 2400 2000 50  0001 C CNN
+	1    2400 2000
+	1    0    0    -1
+$EndComp
+$Comp
+L power:+BATT #PWR0103
+U 1 1 5E172AD1
+P 2400 1800
+F 0 "#PWR0103" H 2400 1650 50  0001 C CNN
+F 1 "+BATT" H 2415 1973 50  0000 C CNN
+F 2 "" H 2400 1800 50  0001 C CNN
+F 3 "" H 2400 1800 50  0001 C CNN
+	1    2400 1800
+	1    0    0    -1
+$EndComp
+Wire Wire Line
+	2400 1800 2500 1800
+Wire Wire Line
+	2400 2000 2500 2000
+Wire Wire Line
+	2300 1900 2500 1900
 $EndSCHEMATC
