File: hardware/pcb/syscon.sch (KiCad schematic (older format))
At the start: 42 parts, among them U100 XC6SLX16-FTG256, U101 W25Q32JVZP, U102 STM32L052K8Ux, U103 PCA9306, X100 24.576MHz, Y100 Crystal

Commit message: pcb: working on ram/ lcd routing
Parts:
- U103: footprint (none) -> Package_SO:VSSOP-8_2.3x2mm_P0.5mm
Changed lines of the file:
@@
 F 0 "U103" H 10150 1500 50  0000 C CNN
 F 1 "PCA9306" H 10100 1400 50  0000 C CNN
-F 2 "" H 9950 2350 50  0001 C CNN
+F 2 "Package_SO:VSSOP-8_2.3x2mm_P0.5mm" H 9950 2350 50  0001 C CNN
 F 3 "http://www.ti.com/lit/ds/symlink/pca9306.pdf" H 10050 2450 50  0001 C CNN
 	1    10350 2000
@@
 $EndComp
 $Comp
-L power:+3V3 #PWR?
+L power:+3V3 #PWR0110
 U 1 1 5E497C1B
 P 9950 1200
-F 0 "#PWR?" H 9950 1050 50  0001 C CNN
+F 0 "#PWR0110" H 9950 1050 50  0001 C CNN
 F 1 "+3V3" H 9965 1373 50  0000 C CNN
 F 2 "" H 9950 1200 50  0001 C CNN
@@
 $EndComp
 $Comp
-L power:+1V8 #PWR?
+L power:+1V8 #PWR0111
 U 1 1 5E4994EF
 P 10450 1500
-F 0 "#PWR?" H 10450 1350 50  0001 C CNN
+F 0 "#PWR0111" H 10450 1350 50  0001 C CNN
 F 1 "+1V8" H 10465 1673 50  0000 C CNN
 F 2 "" H 10450 1500 50  0001 C CNN
@@
 	9400 2100 9950 2100
 $Comp
-L power:GND #PWR?
+L power:GND #PWR0112
 U 1 1 5E4ADA5C
 P 10350 2500
-F 0 "#PWR?" H 10350 2250 50  0001 C CNN
+F 0 "#PWR0112" H 10350 2250 50  0001 C CNN
 F 1 "GND" H 10355 2327 50  0000 C CNN
 F 2 "" H 10350 2500 50  0001 C CNN
@@
 $EndComp
 $Comp
-L power:GND #PWR?
+L power:GND #PWR0113
 U 1 1 5E4B04FB
 P 9750 1500
-F 0 "#PWR?" H 9750 1250 50  0001 C CNN
+F 0 "#PWR0113" H 9750 1250 50  0001 C CNN
 F 1 "GND" H 9755 1327 50  0000 C CNN
 F 2 "" H 9750 1500 50  0001 C CNN
